File: OpenSensor/Hardware/opensenceesp32/opensenceesp32.kicad_pcb (KiCad board)
At the start: 4 copper layers, 22.9 x 73 mm, 20 parts, among them J1 Conn_01x08, Q1 AO3400A, Q2 AO3400A, SW1 SW_Push, SW2 SW_Push_Open, U1 L80-R, U2 LM1117DT-3.3, U3 LM1117DT-5.0, U4 ESP32_C3_OLED

Commit message: First draft of board
Parts:
- added J2: Conn_01x02, Connector_PinSocket_2.54mm:PinSocket_1x02_P2.54mm_Vertical, F.Cu at (242.6, 102.6)
- Q1, Q2, R5, R6, R7, R8: moved to F.Cu
- moved R1 53.6 mm to (218.6, 119.4), turned to 90 degrees
- moved SW1 46.0 mm to (217.7, 64.1), turned to 0 degrees
- moved R7 38.6 mm to (233.7, 65.6), turned to 180 degrees
- moved SW2 38.2 mm to (243.3, 72.0), turned to 180 degrees
- moved R5 32.7 mm to (227.6, 65.7)
- moved R8 29.7 mm to (217.4, 73.2), turned to 90 degrees
- moved R6 24.0 mm to (227.6, 69.3)
- moved Q2 23.4 mm to (223.2, 92.4), turned to 90 degrees
- moved R3 20.2 mm to (222.2, 97.3), turned to 90 degrees
- moved R4 13.8 mm to (227.0, 81.8)
- moved Q1 10.2 mm to (222.5, 119.8), turned to 0 degrees
- moved U1 5.84 mm to (235.7, 120.6)
- moved J1 4.02 mm to (217.8, 89.5)
- moved U2 2.45 mm to (231.1, 94.4)
- moved U3 2.45 mm to (231.1, 103.3)
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Routing:
- net /1PPS: track 0.00 -> 70.4 mm, vias 0 -> 2
- net /SCL: track 0.00 -> 57.1 mm
- net /GPS_TX: track 0.00 -> 53.2 mm, vias 0 -> 1
- net /GPS_RX: track 0.00 -> 48.9 mm, vias 0 -> 1
- net /SDA: track 0.00 -> 47.6 mm
- net Net-(Q1-G): track 0.00 -> 43.1 mm, vias 0 -> 2
- net /GPS_RESET: track 0.00 -> 42.2 mm, vias 0 -> 1
- net +5V: track 0.00 -> 31.7 mm
- net Net-(Q2-G): track 0.00 -> 21.8 mm
- net /L80_GND_SW: track 0.00 -> 21.6 mm
- net /GY_87_GND_SW: track 0.00 -> 19.5 mm
- net GND: track 0.00 -> 18.5 mm, vias 0 -> 9
- net +3.3V: track 0.00 -> 16.5 mm, vias 0 -> 7
- net Net-(U4-GPIO10): track 0.00 -> 15.2 mm
- net VCC: track 0.00 -> 8.81 mm
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- added copper zone on In1.Cu, net +3.3V
- added copper zone on In2.Cu, net GND
- removed copper zone on In1.Cu, net GND
Other:
- board size 22.9 x 73 mm -> 31.8 x 73 mm
