File: Esp32RaymarineSeatalk/ESP32Seatalk/ESP32Seatalk.kicad_sch (KiCad schematic)
At the start: 20 parts, among them J1 SeatalkA, J2 SeatalkB, J3 CAN, J4 CANTRX, J5 GPIO2, J6 GPIO1, J7 GND, Q1 BSS138, U1 AMS1117-3.3, U2 ESP32_C3_OLED

Commit message: ESP32Seatalk hardware: KiCad project updates
Schematic and PCB edits (uncommitted since 2026-09-28), plus project settings: the ERC
pin_to_pin check is now an error and the U3 SW / BST nets are in the Power net class.

Co-Authored-By: Claude Sonnet 5.5 <noreply@anthropic.com>
Parts:
- removed U1: AMS1117-3.3, Package_TO_SOT_SMD:SOT-223-3_TabPin2, symbol Regulator_Linear:AMS1117-3.3
- added C5: 100nf, Capacitor_SMD:C_0805_2012Metric_Pad1.18x1.45mm_HandSolder, symbol Device:C
- added C6: 22uf, Capacitor_Tantalum_SMD:CP_EIA-3216-12_Kemet-S_HandSolder, symbol Device:C_Polarized
- added C7: 100pf, Capacitor_SMD:C_0805_2012Metric_Pad1.18x1.45mm_HandSolder, symbol Device:C
- added L1: 3.3uh, symbol Device:L
- added R3: 31.6k, Resistor_SMD:R_0805_2012Metric_Pad1.20x1.40mm_HandSolder, symbol Device:R
- added R4: 10k, Resistor_SMD:R_0805_2012Metric_Pad1.20x1.40mm_HandSolder, symbol Device:R
- added U3: AP62200, Package_TO_SOT_SMD:SOT-563, symbol Mine9.0:AP62200
- C1: value 4.7u -> 10u
- C3: value 4.7u -> 22uf
Connections:
- net +12V: now also U3.1 (VIN)
- net +3.3V: now also C6.2, C7.1, L1.2, R3.1
- net GND: now also C6.1, R4.2, U3.3 (GND)
- new net: C5.1, U3.4 (BST)
- new net: C5.2, L1.1, U3.2 (SW)
- new net: C7.2, R3.2, R4.1, U3.6 (FB)

Commit message: Seatalk daughter board v2: AP62200 buck, 4-layer, routed, DRC clean, v2 gerbers
Schematic: AMS1117 replaced by AP62200 buck (Cyntec VCHA042A 3.3uH, 0805 ceramics),
custom L1 footprint. Board: 4 layers (In1 +3.3V, In2 GND), hand-routed, KiCad DRC with
schematic parity clean. Gerbers/drill in jlcpcb-export-v2 (v1 export untouched), design
notes and datasheets added.

Co-Authored-By: Claude Sonnet 5.5 <noreply@anthropic.com>
Parts:
- removed C1: 10u, Capacitor_Tantalum_SMD:CP_EIA-3216-12_Kemet-S_HandSolder, symbol Device:C_Polarized
- removed C3, C6: 22uf, Capacitor_Tantalum_SMD:CP_EIA-3216-12_Kemet-S_HandSolder, symbol Device:C_Polarized
- added C1, C3, C6: 22uf, Capacitor_SMD:C_0805_2012Metric_Pad1.18x1.45mm_HandSolder, symbol Device:C
- C4: value 100n -> 22uf
- L1: footprint (none) -> Seatalk-custom:L_Cyntec_VCHA042A-MS6
Connections:
- net +12V: now also C4.1, C3.1
- net +3.3V: now also C1.2, C6.2; no longer C4.2
- net GND: now also C4.2, C1.1, C3.2, C6.1; no longer C4.1
